Commit message: Update robot structure

File: src/amr_description/urdf/amr.urdf.xacro (robot description, xacro)
@@ -1,22 +1,34 @@
 <?xml version="1.0"?>
-<robot name="amr_robot" xmlns:xacro="http://www.ros.org/wiki/xacro">
+<robot xmlns:xacro="http://www.ros.org/wiki/xacro" name="amr">
   <!-- ==================================================== -->
-  <!-- Food Delivery AMR - Master URDF / Xacro Assembly     -->
+  <!-- Core Modular Libraries                               -->
   <!-- ==================================================== -->
-  <!-- Analytical & Helper Macros -->
-  <xacro:include filename="$(find amr_description)/urdf/macros_inertia.xacro"/>
-  <!-- Calibrated Geometric & Mass Properties -->
-  <xacro:include filename="$(find amr_description)/urdf/properties.xacro"/>
-  <!-- Material & Visual Appearance Palette -->
-  <xacro:include filename="$(find amr_description)/urdf/materials.xacro"/>
-  <!-- Base Footprint, Base Link & Chassis Assembly -->
-  <xacro:include filename="$(find amr_description)/urdf/chassis.xacro"/>
-  <!-- Active Differential Drive Wheels -->
-  <xacro:include filename="$(find amr_description)/urdf/drive_wheels.xacro"/>
-  <!-- Passive Caster Wheels Cluster (4x Casters) -->
-  <xacro:include filename="$(find amr_description)/urdf/caster_wheels.xacro"/>
-  <!-- Sensor Links: RPLIDAR A2 & BNO055 IMU -->
-  <xacro:include filename="$(find amr_description)/urdf/sensors.xacro"/>
-  <!-- Gazebo Simulation Plugins & Physics Properties -->
-  <xacro:include filename="$(find amr_description)/urdf/gazebo.xacro"/>
+  <xacro:include filename="properties.xacro" />
+  <xacro:include filename="materials.xacro" />
+  <xacro:include filename="macros_inertia.xacro" />
+  <!-- ==================================================== -->
+  <!-- REP-105 Root Frames: base_footprint & base_link      -->
+  <!-- ==================================================== -->
+  <!-- base_footprint: 2D projection on ground surface (Z = 0) -->
+  <link name="base_footprint"/>
+  <!-- base_link: Center of rotation on active drive axle (Z = wheel_radius = 0.075m) -->
+  <joint name="base_footprint_joint" type="fixed">
+    <parent link="base_footprint"/>
+    <child link="base_link"/>
+    <origin xyz="0 0 ${wheel_radius}" rpy="0 0 0"/>
+  </joint>
+  <link name="base_link"/>
+  <!-- ==================================================== -->
+  <!-- Robot Structural Components                          -->
+  <!-- ==================================================== -->
+  <xacro:include filename="chassis.xacro" />
+  <xacro:include filename="drive_wheels.xacro" />
+  <xacro:include filename="caster_wheels.xacro" />
+  <xacro:include filename="food_trays.xacro" />
+  <xacro:include filename="lidar.xacro" />
+  <xacro:include filename="imu.xacro" />
+  <!-- ==================================================== -->
+  <!-- Gazebo Simulation Plugins & Encoder Feedback         -->
+  <!-- ==================================================== -->
+  <xacro:include filename="gazebo.xacro" />
 </robot>

File: src/amr_description/urdf/caster_wheels.xacro (robot description, xacro)
@@ -2,5 +2,5 @@
 <robot xmlns:xacro="http://www.ros.org/wiki/xacro">
   <!-- ==================================================== -->
-  <!-- Passive Caster Wheel Macro (Frictionless Sphere)    -->
+  <!-- Passive Caster Wheel Macro (Frictionless Sphere)     -->
   <!-- ==================================================== -->
   <xacro:macro name="caster_wheel" params="prefix x_pos y_pos">
@@ -11,11 +11,13 @@
     </joint>
     <link name="caster_${prefix}_link">
+      <!-- Visual: passive_wheel.stl centered at caster rotation center -->
       <visual>
         <origin xyz="-0.0631 1.5650 -0.0335" rpy="${pi/2} 0 0"/>
         <geometry>
-          <mesh filename="package://amr_description/meshes/visual/caster_wheel.stl" scale="1 1 1"/>
+          <mesh filename="package://amr_description/meshes/visual/passive_wheel.stl" scale="1 1 1"/>
         </geometry>
         <material name="robot_caster"/>
       </visual>
+      <!-- Collision: Analytical Sphere for omnidirectional rolling without jamming -->
       <collision>
         <origin xyz="0 0 0" rpy="0 0 0"/>
@@ -24,9 +26,10 @@
         </geometry>
       </collision>
+      <!-- Inertial: Analytical Sphere Inertia -->
       <xacro:inertial_sphere mass="${caster_mass}" radius="${caster_radius}">
         <origin xyz="0 0 0" rpy="0 0 0"/>
       </xacro:inertial_sphere>
     </link>
-    <!-- Gazebo physics: 0 friction ensures smooth omnidirectional sliding without jamming -->
+    <!-- Gazebo physics: Zero friction ensures smooth omnidirectional sliding -->
     <gazebo reference="caster_${prefix}_link">
       <material>Gazebo/Grey</material>
@@ -37,5 +40,5 @@
     </gazebo>
   </xacro:macro>
-  <!-- Instantiate 4 Casters according to Capstone Specs (L = 0.33m, Spacing = 0.40m -> y = +/- 0.20m) -->
+  <!-- Instantiate 4 Casters from defined parametric offsets -->
   <xacro:caster_wheel prefix="fl" x_pos="${caster_x_offset}"  y_pos="${caster_y_offset}"/>
   <xacro:caster_wheel prefix="fr" x_pos="${caster_x_offset}"  y_pos="-${caster_y_offset}"/>

File: src/amr_description/urdf/chassis.xacro (robot description, xacro)
@@ -2,17 +2,5 @@
 <robot xmlns:xacro="http://www.ros.org/wiki/xacro">
   <!-- ==================================================== -->
-  <!-- Base Footprint & Base Link (REP-105 Compliant)       -->
-  <!-- ==================================================== -->
-  <!-- base_footprint: 2D projection on ground surface (z = 0) -->
-  <link name="base_footprint"/>
-  <!-- base_link: Center of rotation on active drive axle -->
-  <joint name="base_footprint_joint" type="fixed">
-    <parent link="base_footprint"/>
-    <child link="base_link"/>
-    <origin xyz="0 0 ${wheel_radius}" rpy="0 0 0"/>
-  </joint>
-  <link name="base_link"/>
-  <!-- ==================================================== -->
-  <!-- Chassis Body Link (Visual Meshes & Analytical Physics) -->
+  <!-- Base Chassis Plate (Centered at X=0, Y=0, Z_ground=40mm) -->
   <!-- ==================================================== -->
   <joint name="chassis_joint" type="fixed">
@@ -22,136 +10,26 @@
   </joint>
   <link name="chassis_link">
-    <!-- Visual 1: Main Base Chassis Structure -->
+    <!-- Visual: Base Chassis Plate STL -->
     <visual>
-      <origin xyz="-0.38 -0.30 -0.04" rpy="${pi/2} 0 ${pi/2}"/>
+      <origin xyz="${-chassis_length/2.0} ${-chassis_width/2.0} ${chassis_z_offset}" rpy="${pi/2} 0 ${pi/2}"/>
       <geometry>
         <mesh filename="package://amr_description/meshes/visual/chassis.stl" scale="1 1 1"/>
       </geometry>
-      <material name="robot_white"/>
-    </visual>
-    <!-- Visual 2: Exterior Body Housing -->
-    <visual>
-      <origin xyz="-0.38 -0.30 -0.04" rpy="${pi/2} 0 ${pi/2}"/>
-      <geometry>
-        <mesh filename="package://amr_description/meshes/visual/housing.stl" scale="1 1 1"/>
-      </geometry>
-      <material name="robot_accent"/>
-    </visual>
-    <!-- Visual 3: Top Cover -->
-    <visual>
-      <origin xyz="-0.38 -0.30 0.15" rpy="0 0 0"/>
-      <geometry>
-        <mesh filename="package://amr_description/meshes/visual/top_cover.stl" scale="1 1 1"/>
-      </geometry>
-      <material name="robot_white"/>
-    </visual>
-    <!-- Visual 4: Food Delivery Trays (3 Tiers - Exactly Centered at X=0, Y=0) -->
-    <!-- Tier 1 Tray -->
-    <visual>
-      <origin xyz="0.360 -0.1825 0.30" rpy="0 0 ${pi/2}"/>
-      <geometry>
-        <mesh filename="package://amr_description/meshes/visual/tray.stl" scale="1 1 1"/>
-      </geometry>
       <material name="robot_metal"/>
     </visual>
-    <!-- Tier 2 Tray -->
-    <visual>
-      <origin xyz="0.360 -0.1825 0.52" rpy="0 0 ${pi/2}"/>
+    <!-- Collision: Analytical Box Plate -->
+    <collision>
+      <origin xyz="0 0 ${chassis_z_offset + chassis_thickness/2.0}" rpy="0 0 0"/>
       <geometry>
-        <mesh filename="package://amr_description/meshes/visual/tray.stl" scale="1 1 1"/>
-      </geometry>
-      <material name="robot_metal"/>
-    </visual>
-    <!-- Tier 3 Tray -->
-    <visual>
-      <origin xyz="0.360 -0.1825 0.74" rpy="0 0 ${pi/2}"/>
-      <geometry>
-        <mesh filename="package://amr_description/meshes/visual/tray.stl" scale="1 1 1"/>
-      </geometry>
-      <material name="robot_metal"/>
-    </visual>
-    <!-- Visual 5: Screen / Head Mount (Thickness scaled to exactly 150mm to match skeleton) -->
-    <visual>
-      <origin xyz="0.075 -0.195 0.904" rpy="0 0 ${pi/2}"/>
-      <geometry>
-        <mesh filename="package://amr_description/meshes/visual/head.stl" scale="1.0 0.9721 1.0"/>
-      </geometry>
-      <material name="robot_dark"/>
-    </visual>
-    <!-- ================================================================= -->
-    <!-- Parametric Offset for Side Assemblies (Wheel Covers, Skeletons, Spacers) -->
-    <!-- Adjust this property to translate both side assemblies inward (+) or outward (-) -->
-    <!-- E.g., value="0.0" is nominal CAD baseline, value="0.0155" retracts inward by 15.5mm -->
-    <!-- ================================================================= -->
-    <xacro:property name="side_inward_offset" value="0.0155"/>
-    <!-- Outward thickness expansion for wheel covers (default: 0.060 = 60mm) -->
-    <!-- Inner mating face against skeleton stays fixed while outer face expands outward -->
-    <xacro:property name="wheel_cover_extra_thickness" value="0.060"/>
-    <!-- Visual 6: Wheel Covers (Inverted U-arch over Drive Wheels) -->
-    <!-- Left Wheel Cover -->
-    <visual>
-      <origin xyz="-0.132 ${0.241 - side_inward_offset + wheel_cover_extra_thickness} -0.03" rpy="${pi/2} 0 0"/>
-      <geometry>
-        <mesh filename="package://amr_description/meshes/visual/wheel_cover.stl" scale="1.0 1.0 ${(0.083 + wheel_cover_extra_thickness) / 0.083}"/>
-      </geometry>
-      <material name="robot_dark"/>
-    </visual>
-    <!-- Right Wheel Cover -->
-    <visual>
-      <origin xyz="0.132 ${-(0.241 - side_inward_offset + wheel_cover_extra_thickness)} -0.03" rpy="${pi/2} 0 ${pi}"/>
-      <geometry>
-        <mesh filename="package://amr_description/meshes/visual/wheel_cover.stl" scale="1.0 1.0 ${(0.083 + wheel_cover_extra_thickness) / 0.083}"/>
-      </geometry>
-      <material name="robot_dark"/>
-    </visual>
-    <!-- Visual 7: Skeleton Pillars (Vertical Frame) -->
-    <!-- Left Skeleton Pillar -->
-    <visual>
-      <origin xyz="-0.101 ${0.398 - side_inward_offset} 0.905" rpy="${pi} 0 0"/>
-      <geometry>
-        <mesh filename="package://amr_description/meshes/visual/skeleton.stl" scale="1 1 1"/>
-      </geometry>
-      <material name="robot_metal"/>
-    </visual>
-    <!-- Right Skeleton Pillar -->
-    <visual>
-      <origin xyz="0.101 ${-(0.398 - side_inward_offset)} 0.905" rpy="0 ${pi} 0"/>
-      <geometry>
-        <mesh filename="package://amr_description/meshes/visual/skeleton.stl" scale="1 1 1"/>
-      </geometry>
-      <material name="robot_metal"/>
-    </visual>
-    <!-- Visual 8: Spacers (Positioned with Skeleton) -->
-    <!-- Left Spacer -->
-    <visual>
-      <origin xyz="-0.101 ${0.398 - side_inward_offset} 0.905" rpy="${pi} 0 0"/>
-      <geometry>
-        <mesh filename="package://amr_description/meshes/visual/spacer.stl" scale="1 1 1"/>
-      </geometry>
-      <material name="robot_dark"/>
-    </visual>
-    <!-- Right Spacer -->
-    <visual>
-      <origin xyz="0.101 ${-(0.398 - side_inward_offset)} 0.905" rpy="0 ${pi} 0"/>
-      <geometry>
-        <mesh filename="package://amr_description/meshes/visual/spacer.stl" scale="1 1 1"/>
-      </geometry>
-      <material name="robot_dark"/>
-    </visual>
-    <!-- Collision Geometry: Simple Analytical Box for High Performance & Zero-Jitter Physics -->
-    <collision>
-      <origin xyz="0 0 0.45" rpy="0 0 0"/>
-      <geometry>
-        <box size="${chassis_length} ${chassis_width} 0.90"/>
+        <box size="${chassis_length} ${chassis_width} ${chassis_thickness}"/>
       </geometry>
     </collision>
-    <!-- Analytical Inertia: Strictly Positive Definite (Prevents Gazebo NaN explosions) -->
-    <xacro:inertial_box mass="${base_mass}" x="${chassis_length}" y="${chassis_width}" z="0.90">
-      <origin xyz="${com_x} ${com_y} ${com_z}" rpy="0 0 0"/>
+    <!-- Inertial: Analytical Box Inertia (${chassis_mass}kg steel/aluminum plate) -->
+    <xacro:inertial_box mass="${chassis_mass}" x="${chassis_length}" y="${chassis_width}" z="${chassis_thickness}">
+      <origin xyz="0 0 ${chassis_z_offset + chassis_thickness/2.0}" rpy="0 0 0"/>
     </xacro:inertial_box>
   </link>
-  <!-- Gazebo Material Settings for Chassis -->
   <gazebo reference="chassis_link">
-    <material>Gazebo/White</material>
+    <material>Gazebo/Grey</material>
   </gazebo>
 </robot>

File: src/amr_description/urdf/drive_wheels.xacro (robot description, xacro)
@@ -2,5 +2,5 @@
 <robot xmlns:xacro="http://www.ros.org/wiki/xacro">
   <!-- ==================================================== -->
-  <!-- Active Differential Drive Wheels (Calibrated)        -->
+  <!-- Active Differential Drive Wheels                     -->
   <!-- ==================================================== -->
   <!-- Left Drive Wheel -->
@@ -8,8 +8,9 @@
     <parent link="base_link"/>
     <child link="left_wheel_link"/>
-    <origin xyz="0 ${wheel_track/2.0} 0" rpy="0 0 0"/>
+    <origin xyz="0 ${wheel_y_offset} 0" rpy="0 0 0"/>
     <axis xyz="0 1 0"/>
   </joint>
   <link name="left_wheel_link">
+    <!-- Visual: active_wheel.stl centered at wheel rotational center -->
     <visual>
       <origin xyz="-0.075 -0.025 -0.075" rpy="0 0 0"/>
@@ -19,22 +20,32 @@
       <material name="robot_wheel"/>
     </visual>
+    <!-- Collision: Analytical Cylinder aligned along Y-axis -->
     <collision>
-      <origin xyz="0 0 0" rpy="${pi/2.0} 0 0"/>
+      <origin xyz="0 0 0" rpy="${pi/2} 0 0"/>
       <geometry>
         <cylinder radius="${wheel_radius}" length="${wheel_width}"/>
       </geometry>
     </collision>
+    <!-- Inertial: Analytical Cylinder Inertia -->
     <xacro:inertial_cylinder mass="${wheel_mass}" length="${wheel_width}" radius="${wheel_radius}">
-      <origin xyz="0 0 0" rpy="${pi/2.0} 0 0"/>
+      <origin xyz="0 0 0" rpy="${pi/2} 0 0"/>
     </xacro:inertial_cylinder>
   </link>
+  <gazebo reference="left_wheel_link">
+    <material>Gazebo/DarkGrey</material>
+    <mu1 value="1.0"/>
+    <mu2 value="1.0"/>
+    <kp value="10000000.0"/>
+    <kd value="1.0"/>
+  </gazebo>
   <!-- Right Drive Wheel -->
   <joint name="right_wheel_joint" type="continuous">
     <parent link="base_link"/>
     <child link="right_wheel_link"/>
-    <origin xyz="0 -${wheel_track/2.0} 0" rpy="0 0 0"/>
+    <origin xyz="0 -${wheel_y_offset} 0" rpy="0 0 0"/>
     <axis xyz="0 1 0"/>
   </joint>
   <link name="right_wheel_link">
+    <!-- Visual: active_wheel.stl centered at wheel rotational center -->
     <visual>
       <origin xyz="-0.075 -0.025 -0.075" rpy="0 0 0"/>
@@ -44,28 +55,22 @@
       <material name="robot_wheel"/>
     </visual>
+    <!-- Collision: Analytical Cylinder aligned along Y-axis -->
     <collision>
-      <origin xyz="0 0 0" rpy="${pi/2.0} 0 0"/>
+      <origin xyz="0 0 0" rpy="${pi/2} 0 0"/>
       <geometry>
         <cylinder radius="${wheel_radius}" length="${wheel_width}"/>
       </geometry>
     </collision>
+    <!-- Inertial: Analytical Cylinder Inertia -->
     <xacro:inertial_cylinder mass="${wheel_mass}" length="${wheel_width}" radius="${wheel_radius}">
-      <origin xyz="0 0 0" rpy="${pi/2.0} 0 0"/>
+      <origin xyz="0 0 0" rpy="${pi/2} 0 0"/>
     </xacro:inertial_cylinder>
   </link>
-  <!-- Wheel Gazebo Material and Friction Settings -->
-  <gazebo reference="left_wheel_link">
-    <material>Gazebo/DarkGrey</material>
-    <mu1 value="0.6"/>
-    <mu2 value="0.4"/>
-    <kp value="1000000.0"/>
-    <kd value="100.0"/>
-  </gazebo>
   <gazebo reference="right_wheel_link">
     <material>Gazebo/DarkGrey</material>
-    <mu1 value="0.6"/>
-    <mu2 value="0.4"/>
-    <kp value="1000000.0"/>
-    <kd value="100.0"/>
+    <mu1 value="1.0"/>
+    <mu2 value="1.0"/>
+    <kp value="10000000.0"/>
+    <kd value="1.0"/>
   </gazebo>
 </robot>

File: src/amr_description/urdf/gazebo.xacro (robot description, xacro)
@@ -2,33 +2,10 @@
 <robot xmlns:xacro="http://www.ros.org/wiki/xacro">
   <!-- ==================================================== -->
-  <!-- Gazebo Plugins Configuration                         -->
+  <!-- Gazebo Simulation & Hardware Feedback Plugins        -->
   <!-- ==================================================== -->
-  <!-- Differential Drive Controller Plugin -->
-  <gazebo>
-    <plugin name="diff_drive_controller" filename="libgazebo_ros_diff_drive.so">
-      <!-- Update rate in Hz -->
-      <update_rate>50</update_rate>
-      <!-- Wheel joints -->
-      <left_joint>left_wheel_joint</left_joint>
-      <right_joint>right_wheel_joint</right_joint>
-      <!-- Kinematics from Capstone Specifications -->
-      <wheel_separation>${wheel_track}</wheel_separation>
-      <wheel_diameter>${2.0 * wheel_radius}</wheel_diameter>
-      <!-- Limits -->
-      <max_wheel_torque>20</max_wheel_torque>
-      <max_wheel_acceleration>2.0</max_wheel_acceleration>
-      <!-- Output topics -->
-      <command_topic>cmd_vel</command_topic>
-      <odometry_topic>wheel/odom</odometry_topic>
-      <odometry_frame>odom</odometry_frame>
-      <robot_base_frame>base_footprint</robot_base_frame>
-      <!-- Odometry and TF broadcasting -->
-      <publish_odom>true</publish_odom>
-      <!-- EKF (robot_localization) handles odom -> base_footprint transform -->
-      <publish_odom_tf>false</publish_odom_tf>
-      <publish_wheel_tf>true</publish_wheel_tf>
-    </plugin>
-  </gazebo>
-  <!-- Joint State Publisher Plugin -->
+  <!-- Joint State Publisher Plugin (Wheel Encoders Feedback) -->
+  <!-- Publishes sensor_msgs/JointState on /joint_states     -->
+  <!-- Provides angular position (rad -> revolutions) and    -->
+  <!-- angular velocity (rad/s -> RPM) for each drive wheel  -->
   <gazebo>
     <plugin name="joint_state_publisher" filename="libgazebo_ros_joint_state_publisher.so">
@@ -38,53 +15,29 @@
     </plugin>
   </gazebo>
-  <!-- 2D LiDAR Ray Sensor Plugin (Slamtec RPLIDAR A2) -->
-  <gazebo reference="laser_frame">
-    <sensor name="lidar_sensor" type="ray">
-      <pose>0 0 0 0 0 0</pose>
-      <visualize>false</visualize>
-      <update_rate>10</update_rate>
-      <ray>
-        <scan>
-          <horizontal>
-            <samples>800</samples>
-            <resolution>1</resolution>
-            <min_angle>-3.14159265</min_angle>
-            <max_angle>3.14159265</max_angle>
-          </horizontal>
-        </scan>
-        <range>
-          <min>0.20</min>
-          <max>12.0</max>
-          <resolution>0.01</resolution>
-        </range>
-        <noise>
-          <type>gaussian</type>
-          <mean>0.0</mean>
-          <stddev>0.01</stddev>
-        </noise>
-      </ray>
-      <plugin name="lidar_controller" filename="libgazebo_ros_ray_sensor.so">
-        <ros>
-          <remapping>~/out:=scan</remapping>
-        </ros>
-        <output_type>sensor_msgs/LaserScan</output_type>
-        <frame_name>laser_frame</frame_name>
-      </plugin>
-    </sensor>
-  </gazebo>
-  <!-- 9-DOF IMU Sensor Plugin (Bosch BNO055) -->
-  <gazebo reference="imu_link">
-    <sensor name="imu_sensor" type="imu">
-      <always_on>true</always_on>
-      <update_rate>100</update_rate>
-      <visualize>false</visualize>
-      <plugin name="imu_controller" filename="libgazebo_ros_imu_sensor.so">
-        <ros>
-          <remapping>~/out:=imu/data</remapping>
-        </ros>
-        <initial_orientation_as_reference>false</initial_orientation_as_reference>
-        <frame_name>imu_link</frame_name>
-      </plugin>
-    </sensor>
+  <!-- Differential Drive Controller Plugin -->
+  <!-- Drives active wheels via /cmd_vel and calculates     -->
+  <!-- odometry integration from wheel encoder feedback     -->
+  <gazebo>
+    <plugin name="diff_drive_controller" filename="libgazebo_ros_diff_drive.so">
+      <update_rate>50</update_rate>
+      <!-- Wheel joints -->
+      <left_joint>left_wheel_joint</left_joint>
+      <right_joint>right_wheel_joint</right_joint>
+      <!-- Kinematic parameters from properties.xacro -->
+      <wheel_separation>${wheel_track}</wheel_separation>
+      <wheel_diameter>${2.0 * wheel_radius}</wheel_diameter>
+      <!-- Dynamic limits -->
+      <max_wheel_torque>20</max_wheel_torque>
+      <max_wheel_acceleration>2.0</max_wheel_acceleration>
+      <!-- Topics & Frames -->
+      <command_topic>cmd_vel</command_topic>
+      <odometry_topic>wheel/odom</odometry_topic>
+      <odometry_frame>odom</odometry_frame>
+      <robot_base_frame>base_footprint</robot_base_frame>
+      <!-- Odometry and TF broadcasting -->
+      <publish_odom>true</publish_odom>
+      <publish_odom_tf>true</publish_odom_tf>
+      <publish_wheel_tf>true</publish_wheel_tf>
+    </plugin>
   </gazebo>
 </robot>
